File: powerBank.kicad_pcb (KiCad board)
At the start: 2 copper layers, 98.4 x 40.6 mm, 9 parts, among them J2 USB_C_Receptacle_PowerOnly_6P

Commit message: Gerber files
Routing:
- net Net-(D1-K): track 67.5 -> 81.3 mm
- net Net-(D1-A): track 49.9 -> 61.0 mm
Changed lines of the file:
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@@
 			(drillshape 0)
 			(scaleselection 1)
-			(outputdirectory "C:/Users/prana/Documents/powerBank/Portable-Charger-PCB/gerbers/")
+			(outputdirectory "C:/Users/prana/Documents/powerBank/Portable-Charger-PCB/gerbersv2/")
 		)
 	)
@@
 			(at 0 -2.85 0)
 			(layer "F.SilkS")
+			(hide yes)
 			(effects
 				(font
@@
 			(at 0 -2.85 0)
 			(layer "F.SilkS")
+			(hide yes)
 			(effects
 				(font
@@
 	)
 	(segment
-		(start 181.565 67.605)
-		(end 189.405 67.605)
-		(width 0.8)
-		(layer "F.Cu")
-		(net 5)
-	)
-	(segment
-		(start 168.525 80.645)
-		(end 181.565 67.605)
-		(width 0.8)
-		(layer "F.Cu")
-		(net 5)
-	)
-	(segment
-		(start 177.8 64.135)
-		(end 181.27 67.605)
-		(width 0.8)
-		(layer "F.Cu")
-		(net 5)
-	)
-	(segment
-		(start 181.27 67.605)
-		(end 181.565 67.605)
-		(width 0.2)
+		(start 181.27 67.65)
+		(end 168.706 80.214)
+		(width 0.8)
 		(layer "F.Cu")
 		(net 5)
@@
 	)
 	(segment
+		(start 193.38 67.605)
+		(end 193.675 67.31)
+		(width 0.8)
+		(layer "F.Cu")
+		(net 5)
+	)
+	(segment
+		(start 193.675 67.31)
+		(end 193.675 64.77)
+		(width 0.8)
+		(layer "F.Cu")
+		(net 5)
+	)
+	(segment
+		(start 181.27 67.605)
+		(end 177.8 64.135)
+		(width 0.8)
+		(layer "F.Cu")
+		(net 5)
+	)
+	(segment
+		(start 193.47 64.565)
+		(end 189.405 64.565)
+		(width 0.8)
+		(layer "F.Cu")
+		(net 5)
+	)
+	(segment
+		(start 181.27 67.605)
+		(end 181.27 67.65)
+		(width 0.8)
+		(layer "F.Cu")
+		(net 5)
+	)
+	(segment
 		(start 184.78 60.96)
 		(end 188.385 64.565)
@@
 	)
 	(segment
-		(start 167.64 70.2775)
-		(end 167.7425 70.175)
+		(start 189.405 67.605)
+		(end 193.38 67.605)
+		(width 0.8)
+		(layer "F.Cu")
+		(net 5)
+	)
+	(segment
+		(start 193.675 64.77)
+		(end 193.47 64.565)
+		(width 0.8)
+		(layer "F.Cu")
+		(net 5)
+	)
+	(segment
+		(start 168.706 80.214)
+		(end 168.706 80.645)
+		(width 0.8)
+		(layer "F.Cu")
+		(net 5)
+	)
+	(segment
+		(start 189.405 67.605)
+		(end 181.27 67.605)
+		(width 0.8)
+		(layer "F.Cu")
+		(net 5)
+	)
+	(segment
+		(start 167.005 86.36)
+		(end 167.64 85.725)
+		(width 0.8)
+		(layer "F.Cu")
+		(net 6)
+	)
+	(segment
+		(start 189.405 70.835)
+		(end 189.405 68.835)
 		(width 0.2)
 		(layer "F.Cu")
@@
 	)
 	(segment
-		(start 167.64 84.455)
-		(end 167.005 83.82)
-		(width 0.8)
+		(start 189.405 63.335)
+		(end 189.405 61.015)
+		(width 0.2)
 		(layer "F.Cu")
 		(net 6)
 	)
 	(segment
-		(start 167.005 83.82)
-		(end 167.005 81.915)
-		(width 0.8)
-		(layer "F.Cu")
-		(net 6)
-	)
-	(segment
-		(start 157.48 71.755)
-		(end 159.06 70.175)
-		(width 0.2)
-		(layer "F.Cu")
-		(net 6)
-	)
-	(segment
-		(start 156.845 71.755)
-		(end 157.48 71.755)
-		(width 0.2)
+		(start 167.64 85.725)
+		(end 167.64 80.645)
+		(width 0.8)
 		(layer "F.Cu")
 		(net 6)
@@
 	)
 	(segment
-		(start 159.06 70.175)
-		(end 167.7425 70.175)
+		(start 189.405 63.335)
+		(end 194.78 63.335)
 		(width 0.8)
 		(layer "F.Cu")
@@
 	)
 	(segment
+		(start 189.46 70.89)
+		(end 189.405 70.835)
+		(width 0.2)
+		(layer "F.Cu")
+		(net 6)
+	)
+	(segment
+		(start 189.405 61.015)
+		(end 189.46 60.96)
+		(width 0.2)
+		(layer "F.Cu")
+		(net 6)
+	)
+	(segment
+		(start 194.945 69.215)
+		(end 194.565 68.835)
+		(width 0.8)
+		(layer "F.Cu")
+		(net 6)
+	)
+	(segment
+		(start 165.735 80.645)
+		(end 156.845 71.755)
+		(width 0.8)
+		(layer "F.Cu")
+		(net 6)
+	)
+	(segment
+		(start 167.64 80.645)
+		(end 165.735 80.645)
+		(width 0.8)
+		(layer "F.Cu")
+		(net 6)
+	)
+	(segment
+		(start 194.565 68.835)
+		(end 189.405 68.835)
+		(width 0.8)
+		(layer "F.Cu")
+		(net 6)
+	)
+	(segment
+		(start 189.46 71.21)
+		(end 193.04 71.21)
+		(width 0.2)
+		(layer "F.Cu")
+		(net 6)
+	)
+	(segment
+		(start 183.26 72.645)
+		(end 169.545 86.36)
+		(width 0.8)
+		(layer "F.Cu")
+		(net 6)
+	)
+	(segment
+		(start 194.78 63.335)
+		(end 194.945 63.5)
+		(width 0.8)
+		(layer "F.Cu")
+		(net 6)
+	)
+	(segment
+		(start 189.46 71.21)
+		(end 189.46 70.89)
+		(width 0.2)
+		(layer "F.Cu")
+		(net 6)
+	)
+	(segment
+		(start 169.545 86.36)
+		(end 167.005 86.36)
+		(width 0.8)
+		(layer "F.Cu")
+		(net 6)
+	)
+	(segment
+		(start 194.945 63.5)
+		(end 194.945 69.215)
+		(width 0.8)
+		(layer "F.Cu")
+		(net 6)
+	)
+	(segment
+		(start 189.46 60.96)
+		(end 193.04 60.96)
+		(width 0.2)
+		(layer "F.Cu")
+		(net 6)
+	)
+	(segment
 		(start 183.26 68.835)
-		(end 167.64 84.455)
-		(width 0.8)
-		(layer "F.Cu")
-		(net 6)
-	)
-	(segment
-		(start 167.64 80.645)
-		(end 167.64 70.2775)
-		(width 0.8)
-		(layer "F.Cu")
-		(net 6)
-	)
-	(segment
-		(start 167.005 81.915)
-		(end 156.845 71.755)
-		(width 0.8)
-		(layer "F.Cu")
+		(end 183.26 72.645)
+		(width 0.8)
+		(layer "F.Cu")
